Commit message: correct structure

File: farmbot_description.urdf (robot description, URDF)
Before this commit: robot farmbot, 10 links, 3 joints
Joints:
- added joint joint4: type fixed, parent link1, child link5
- added joint joint5: type revolute, parent link1, child link10
- added joint joint6: type continuous, parent link2, child link6
- added joint joint7: type continuous, parent link3, child link7
- added joint joint8: type continuous, parent link4, child link8
- added joint joint9: type continuous, parent link5, child link9
- joint joint1: type continuous -> fixed
- joint joint2: type continuous -> fixed
- joint joint3: parent link3 -> link1; type continuous -> fixed

Commit message: correct structure

File: farmbot_description.urdf (robot description, URDF)
Before this commit: robot farmbot, 10 links, 9 joints
Joints:
- joint joint5: axis (none) -> 0 0 1; limit (none) -> lower=-3.1 upper=3.1 effort=0.1 velocity=0.2; origin (none) -> xyz=0 0.25 0 rpy=0 0 0
