Commit message: start of robot budy in urdf file

File: description/urdf/base_link.urdf (robot description, URDF)
Before this commit: robot RoboGardener, 1 links, 0 joints
Links:
- added link wheel_left; visual cylinder length=0.05 radius=0.1
- added link wheel_right; visual cylinder length=0.05 radius=0.1
Joints:
- added joint base_to_left_wheel: type fixed, parent base_link, child wheel_left, origin xyz=0.25 0.25 -0.05 rpy=-1.6 0 0
- added joint base_to_right_wheel: type fixed, parent base_link, child wheel_right, origin xyz=0.25 -0.25 -0.05 rpy=1.6 0 0

Commit message: base of roboter scelette

File: description/urdf/base_link.urdf (robot description, URDF)
Before this commit: robot RoboGardener, 3 links, 2 joints
Links:
- added link motorwheel_left; visual cylinder length=0.05 radius=0.1
- added link motorwheel_right; visual cylinder length=0.05 radius=0.1
Joints:
- added joint base_to_left_motorwheel: type fixed, parent base_link, child motorwheel_left, origin xyz=-0.25 0.25 -0.05 rpy=-1.6 0 0
- added joint base_to_right_motorwheel: type fixed, parent base_link, child motorwheel_right, origin xyz=-0.25 -0.25 -0.05 rpy=1.6 0 0

Commit message: add arms to robot body, test creation of frames pdf

File: description/urdf/base_link.urdf (robot description, URDF)
Before this commit: robot RoboGardener, 5 links, 4 joints
Links:
- added link hand; visual sphere radius=0.04
- added link leftarm; visual cylinder length=0.1 radius=0.02
- added link rightarm; visual cylinder length=0.1 radius=0.02
- added link scissor; visual cylinder length=0.05 radius=0.025
Joints:
- added joint base_to_leftarm: type fixed, parent base_link, child leftarm, origin xyz=0.3 0.15 0 rpy=0 1.6 0
- added joint base_to_rightarm: type fixed, parent base_link, child rightarm, origin xyz=0.3 -0.15 0 rpy=0 1.6 0
- added joint leftarm_to_hand: type fixed, parent leftarm, child hand, origin xyz=0 0 0.05 rpy=0 0 0
- added joint rightarm_to_scissors: type fixed, parent rightarm, child scissor, origin xyz=0 0 0.05 rpy=0 1.6 0
