Commit message: front wheel with arm

File: description/urdf/batmobil.urdf (robot description, URDF)
Before this commit: robot batmobil, 4 links, 3 joints
Links:
- added link front_wheel; visual cylinder length=0.1 radius=0.23
- added link wheel_arm_left; visual box size=0.02 0.03 0.4
- added link wheel_arm_right; visual box size=0.02 0.03 0.23
Joints:
- added joint arm_to_front_wheel: type continuous, parent wheel_arm_left, child front_wheel, origin xyz=0 0 0 rpy=-${pi/2} 0 0, axis 0 -0.25 1
- added joint base_to_wheel_arm_left: type fixed, parent base_link, child wheel_arm_left, origin xyz=-1.5 -0.1 -0.12
- added joint base_to_wheel_arm_right: type fixed, parent base_link, child wheel_arm_right, origin xyz=-1.5 0.1 -0.12

Commit message: add collision

File: description/urdf/batmobil.urdf (robot description, URDF)
Before this commit: robot batmobil, 7 links, 6 joints
Links:
- link chassis: geometry collision box size=2.1 0.95 0.02; visual box size=2.1 0.95 0.02
- link front_wheel: geometry collision cylinder length=0.1 radius=0.13; visual cylinder length=0.1 radius=0.13
- link left_wheel: geometry collision cylinder length=0.24 radius=0.3; visual cylinder length=0.24 radius=0.3
- link right_wheel: geometry collision cylinder length=0.24 radius=0.3; visual cylinder length=0.24 radius=0.3
- link wheel_arm_left: geometry collision box size=0.02 0.03 0.3; visual box size=0.02 0.03 0.3
- link wheel_arm_right: geometry collision box size=0.02 0.03 0.3; visual box size=0.02 0.03 0.3
Joints:
- joint arm_to_front_wheel: axis 0 -0.25 1 -> 0 0 1; origin xyz=0 0 0 rpy=-${pi/2} 0 0 -> xyz=0 0.05 -0.15 rpy=-${pi/2} 0 0
- joint base_to_left_wheel: origin xyz=0 0.475 0 rpy=-${pi/2} 0 0 -> xyz=0 0.475 -0.1 rpy=-${pi/2} 0 0
- joint base_to_right_wheel: origin xyz=0 -0.475 0 rpy=${pi/2} 0 0 -> xyz=0 -0.475 -0.1 rpy=${pi/2} 0 0
- joint base_to_wheel_arm_left: origin xyz=-1.5 -0.1 -0.12 -> xyz=-1.5 -0.05 -0.15
- joint base_to_wheel_arm_right: origin xyz=-1.5 0.1 -0.12 -> xyz=-1.5 0.05 -0.15
