Commit message: correct urdf file for gazebo

File: description/gazebo_sim/batmobil_gz.urdf (robot description, URDF)
Before this commit: robot batmobil, 7 links, 6 joints
Joints:
- joint arm_to_front_wheel: origin xyz=0 0.05 -0.15 rpy=-${pi/2} 0 0 -> xyz=0 0.05 -0.15 rpy=-1.5708 0 0
- joint base_to_left_wheel: origin xyz=0 0.475 -0.1 rpy=-${pi/2} 0 0 -> xyz=0 0.475 -0.1 rpy=-1.5708 0 0
- joint base_to_right_wheel: origin xyz=0 -0.475 -0.1 rpy=${pi/2} 0 0 -> xyz=0 -0.475 -0.1 rpy=1.5708 0 0
