Commit message: add gz, ros2 control, tf2_ros and controller manager node to launch file

File: model/description/core_model.xacro (robot description, xacro)
@@ -21,5 +21,5 @@
     <parent link="dummy_link"/>
     <child link="base_link"/>
-    <origin xyz="0 0 0" rpy="0 0 0"/>
+    <origin xyz="0 0 1" rpy="0 0 0"/>
   </joint>
     <!-- Base Link -->

File: model/description/gz_control.xacro (robot description, xacro)
@@ -4,22 +4,23 @@
         <plugin name="gz::sim::systems::DiffDrive" filename="gz-sim-diff-drive-system">
             <!-- Wheel Information -->
-            <left_joint>base_to_left_wheel</left_joint>
-            <right_joint>base_to_right_wheel</right_joint>
+            <left_joint>left_wheel_joint</left_joint>
+            <right_joint>right_wheel_joint</right_joint>
             <wheel_separation>0.95</wheel_separation>
             <wheel_radius>0.3</wheel_radius>
             <!-- Input -->
-            <topic>cmd_vel</topic>
+            <topic>/cmd_vel</topic>
             <!-- Output -->
             <frame_id>odom</frame_id>
             <child_frame_id>base_link</child_frame_id>
             <odom_topic>odom</odom_topic>
-            <odom_publish_frequency>1</odom_publish_frequency>
-            <tf_topic>/tf</tf_topic>
+            <odom_publish_frequency>50</odom_publish_frequency>
+            <!-- TF Publishing -->
+            <publish_tf>true</publish_tf>
         </plugin>
         <plugin filename="gz-sim-joint-state-publisher-system"
             name="gz::sim::systems::JointStatePublisher">
             <topic>joint_states</topic>
-            <joint_name>base_to_left_wheel</joint_name>
-            <joint_name>base_to_right_wheel</joint_name>
+            <joint_name>left_wheel_joint</joint_name>
+            <joint_name>right_wheel_joint</joint_name>
         </plugin>
     </gazebo>

File: model/description/robo.urdf.xacro (robot description, xacro)
@@ -6,4 +6,5 @@
     <xacro:include filename="core_model.xacro" />
     <xacro:include filename="materials.xacro" />
+    <xacro:include filename="gz_control.xacro" />
     <!-- Macro Invocation -->
     <xacro:robot />
